File: cores/rollerg/sch/Scroll.kicad_sch (KiCad schematic)
At the start: 0 parts

Commit message: wip rollerg sch: objects page
Parts:
- added 12K1, 12L1: 955D05-06-07-08, symbol konami:955D05-06-07-08
- added 13J1: 051962, symbol konami:051962
- added 16J1: 052109, symbol konami:052109
- added 16K1, 16L1: MB8464A-10W-15W, symbol fujitsu:MB8464A-10W-15W
- added H1: 74LS07, symbol 74xx:74LS07
Connections:
- new net: 16J1.98 (~{RST}), H1.9
- new net ACOL0: 13J1.30 (DSB0)
- new net ACOL1: 13J1.32 (DSB1)
- new net ACOL2: 13J1.33 (DSB2)
- new net ACOL3: 13J1.34 (DSB3)
- new net APAL0: 13J1.36 (DSB5)
- new net APAL1: 13J1.37 (DSB6)
- new net APAL2: 13J1.38 (DSB7)
- new net BCOL0: 13J1.46 (DSA0)
- new net BCOL1: 13J1.47 (DSA1)
- new net BCOL2: 13J1.48 (DSA2)
- new net BCOL3: 13J1.49 (DSA3)
- new net BPAL0: 13J1.51 (DSA5)
- new net BPAL1: 13J1.52 (DSA6)
- new net BPAL2: 13J1.53 (DSA7)
- new net COL5: 13J1.109 (COL5), 16J1.42 (COL5)
- new net COL6: 13J1.108 (COL6), 16J1.43 (COL6)
- new net COL7: 13J1.107 (COL7), 16J1.46 (COL7)
- new net FCOL0: 13J1.59 (DFI0)
- new net FCOL1: 13J1.60 (DFI1)
- new net FCOL2: 13J1.62 (DFI2)
- new net FCOL3: 13J1.63 (DFI3)
- new net FPAL0: 13J1.65 (DFI5)
- new net FPAL1: 13J1.66 (DFI6)
- new net FPAL3: 13J1.67 (DFI7)
- new net GFXROMA0: 12K1.9 (A0), 12L1.9 (A0), 16J1.35 (VC0)
- new net GFXROMA1: 12K1.8 (A1), 12L1.8 (A1), 16J1.34 (VC1)
- new net GFXROMA10: 12K1.38 (A10), 12L1.38 (A10), 16J1.24 (VC10)
- new net GFXROMA11: 12K1.37 (A11), 12L1.37 (A11), 16J1.37 (COL0)
- new net GFXROMA12: 12K1.36 (A12), 12L1.36 (A12), 16J1.38 (COL1)
- new net GFXROMA13: 12K1.35 (A13), 12L1.35 (A13), 16J1.41 (COL4)
- new net GFXROMA14: 12K1.34 (A14), 12L1.34 (A14), 16J1.39 (COL2)
- new net GFXROMA15: 12K1.33 (A15), 12L1.33 (A15), 16J1.40 (COL3)
- new net GFXROMA16: 12K1.32 (A16), 12L1.32 (A16), 16J1.23 (CAB1)
- new net GFXROMA17: 12K1.1 (A17), 12L1.1 (A17), 16J1.22 (CAB2)
- new net GFXROMA2: 12K1.7 (A2), 12L1.7 (A2), 16J1.33 (VC2)
- new net GFXROMA3: 12K1.6 (A3), 12L1.6 (A3), 16J1.32 (VC3)
- new net GFXROMA4: 12K1.5 (A4), 12L1.5 (A4), 16J1.30 (VC4)
- new net GFXROMA5: 12K1.4 (A5), 12L1.4 (A5), 16J1.29 (VC5)
- new net GFXROMA6: 12K1.3 (A6), 12L1.3 (A6), 16J1.28 (VC6)
- new net GFXROMA7: 12K1.2 (A7), 12L1.2 (A7), 16J1.27 (VC7)
- new net GFXROMA8: 12K1.40 (A8), 12L1.40 (A8), 16J1.26 (VC8)
- new net GFXROMA9: 12K1.39 (A9), 12L1.39 (A9), 16J1.25 (VC9)
- new net GFXROMD0: 12L1.13 (D0), 13J1.29 (VC0)
- new net GFXROMD1: 12L1.15 (D1), 13J1.28 (VC1)
- new net GFXROMD10: 12L1.18 (D10), 13J1.19 (VC10)
- new net GFXROMD11: 12L1.20 (D11), 13J1.18 (VC11)
- new net GFXROMD12: 12L1.23 (D12), 13J1.17 (VC12)
- new net GFXROMD13: 12L1.25 (D13), 13J1.16 (VC13)
- new net GFXROMD14: 12L1.27 (D14), 13J1.13 (VC14)
- new net GFXROMD15: 12L1.29 (D15/A-1), 13J1.12 (VC15)
- new net GFXROMD16: 12K1.13 (D0), 13J1.11 (VC16)
- new net GFXROMD17: 12K1.15 (D1), 13J1.10 (VC17)
- new net GFXROMD18: 12K1.17 (D2), 13J1.9 (VC18)
- new net GFXROMD19: 12K1.19 (D3), 13J1.8 (VC19)
- new net GFXROMD2: 12L1.17 (D2), 13J1.27 (VC2)
- new net GFXROMD20: 12K1.22 (D4), 13J1.7 (VC20)
- new net GFXROMD21: 12K1.24 (D5), 13J1.6 (VC21)
- new net GFXROMD22: 12K1.26 (D6), 13J1.5 (VC22)
- new net GFXROMD23: 12K1.28 (D7), 13J1.4 (VC23)
- new net GFXROMD24: 12K1.14 (D8), 13J1.3 (VC24)
- new net GFXROMD25: 12K1.16 (D9), 13J1.2 (VC25)
- new net GFXROMD26: 12K1.18 (D10), 13J1.120 (VC26)
- new net GFXROMD27: 12K1.20 (D11), 13J1.119 (VC27)
- new net GFXROMD28: 12K1.23 (D12), 13J1.118 (VC28)
- new net GFXROMD29: 12K1.25 (D13), 13J1.117 (VC29)
- new net GFXROMD3: 12L1.19 (D3), 13J1.26 (VC3)
- new net GFXROMD30: 12K1.27 (D14), 13J1.116 (VC30)
- new net GFXROMD31: 12K1.29 (D15/A-1), 13J1.115 (VC31)
- new net GFXROMD4: 12L1.22 (D4), 13J1.25 (VC4)
- new net GFXROMD5: 12L1.24 (D5), 13J1.24 (VC5)
- new net GFXROMD6: 12L1.26 (D6), 13J1.23 (VC6)
- new net GFXROMD7: 12L1.28 (D7), 13J1.22 (VC7)
- new net GFXROMD8: 12L1.14 (D8), 13J1.21 (VC8)
- new net GFXROMD9: 12L1.16 (D9), 13J1.20 (VC9)
- new net M12: 13J1.95 (M12)
- new net M6: 13J1.78 (M6)
- new net MAIN_A1: 13J1.88 (AB0), 16J1.66 (AB0)
- new net MAIN_A10: 16J1.111 (AB9)
- new net MAIN_A11: 16J1.110 (AB10)
- new net MAIN_A13: 16J1.109 (AB11)
- new net MAIN_A14: 16J1.80 (AB12)
- new net MAIN_A15: 16J1.82 (AB14)
- new net MAIN_A16: 16J1.83 (AB15)
- new net MAIN_A2: 13J1.89 (AB1), 16J1.67 (AB1)
- new net MAIN_A3: 16J1.68 (AB2)
- new net MAIN_A4: 16J1.69 (AB3)
- new net MAIN_A5: 16J1.116 (AB4)
- new net MAIN_A6: 16J1.115 (AB5)
- new net MAIN_A7: 16J1.114 (AB6)
- new net MAIN_A8: 16J1.113 (AB7)
- new net MAIN_A9: 16J1.112 (AB8)
- new net MAIN_DB0: 13J1.79 (DB0), 16J1.56 (DB0)
- new net MAIN_DB1: 13J1.80 (DB1), 16J1.57 (DB1)
- new net MAIN_DB2: 13J1.81 (DB2), 16J1.58 (DB2)
- new net MAIN_DB3: 13J1.82 (DB3), 16J1.59 (DB3)
- new net MAIN_DB4: 13J1.83 (DB4), 16J1.60 (DB4)
- new net MAIN_DB5: 13J1.84 (DB5), 16J1.62 (DB5)
- new net MAIN_DB6: 13J1.85 (DB6), 16J1.63 (DB6)
- new net MAIN_DB7: 13J1.86 (DB7), 16J1.64 (DB7)
- new net M~{RD}: 13J1.87 (~{RD}), 16J1.85 (~{RD})
- new net PE: 16J1.90 (PE)
- new net PQ: 16J1.89 (PQ)
- new net RM~{RD}: 13J1.96 (RM~{RD}), 16J1.97 (RM~{RD})
- new net SCRAMA0: 16J1.2 (RA0), 16K1.10 (A0), 16L1.10 (A0)
- new net SCRAMA1: 16J1.120 (RA1), 16K1.9 (A1), 16L1.9 (A1)
- new net SCRAMA10: 16J1.77 (RA10), 16K1.21 (A10), 16L1.21 (A10)
- new net SCRAMA11: 16J1.78 (RA11), 16K1.23 (A11), 16L1.23 (A11)
- new net SCRAMA12: 16J1.79 (RA12), 16K1.2 (A12), 16L1.2 (A12)
- new net SCRAMA2: 16J1.119 (RA2), 16K1.8 (A2), 16L1.8 (A2)
- new net SCRAMA3: 16J1.118 (RA3), 16K1.7 (A3), 16L1.7 (A3)
- new net SCRAMA4: 16J1.117 (RA4), 16K1.6 (A4), 16L1.6 (A4)
- new net SCRAMA5: 16J1.70 (RA5), 16K1.5 (A5), 16L1.5 (A5)
- new net SCRAMA6: 16J1.71 (RA6), 16K1.4 (A6), 16L1.4 (A6)
- new net SCRAMA7: 16J1.72 (RA7), 16K1.3 (A7), 16L1.3 (A7)
- new net SCRAMA8: 16J1.73 (RA8), 16K1.25 (A8), 16L1.25 (A8)
- new net SCRAMA9: 16J1.76 (RA9), 16K1.24 (A9), 16L1.24 (A9)
- new net SCR~{CLK}: 13J1.90 (M24), 16J1.65 (M24)
- new net VCC: 12K1.21 (VCC), 12K1.31 (BYTE), 12L1.21 (VCC), 12L1.31 (BYTE), 13J1.104 (VCC), 13J1.14 (VCC), 13J1.44 (VCC), 13J1.74 (VCC), 16J1.104 (VCC), 16J1.14 (VCC), 16J1.44 (VCC), 16J1.74 (VCC), 16K1.26 (~{CS2}), 16K1.28 (VCC), 16L1.26 (~{CS2}), 16L1.28 (VCC)
- new net VD0: 16J1.20 (VD0), 16K1.11 (D0)
- new net VD1: 16J1.19 (VD1), 16K1.12 (D1)
- new net VD10: 16J1.8 (VD10), 16L1.13 (D2)
- new net VD11: 16J1.7 (VD11), 16L1.15 (D3)
- new net VD12: 16J1.6 (VD12), 16L1.16 (D4)
- new net VD13: 16J1.5 (VD13), 16L1.17 (D5)
- new net VD14: 16J1.4 (VD14), 16L1.18 (D6)
- new net VD15: 16J1.3 (VD15), 16L1.19 (D7)
- new net VD2: 16J1.18 (VD2), 16K1.13 (D2)
- new net VD3: 16J1.17 (VD3), 16K1.15 (D3)
- new net VD4: 16J1.16 (VD4), 16K1.16 (D4)
- new net VD5: 16J1.13 (VD5), 16K1.17 (D5)
- new net VD6: 16J1.12 (VD6), 16K1.18 (D6)
- new net VD7: 16J1.11 (VD7), 16K1.19 (D7)
- new net VD8: 16J1.10 (VD8), 16L1.11 (D0)
- new net VD9: 16J1.9 (VD9), 16L1.12 (D1)
- new net VSS: 12K1.10 (~{CE}), 12K1.11 (VSS), 12K1.12 (~{OE}), 12K1.30 (VSS), 12L1.10 (~{CE}), 12L1.11 (VSS), 12L1.12 (~{OE}), 12L1.30 (VSS), 13J1.1 (VSS), 13J1.105 (VSS), 13J1.110 (COL4), 13J1.111 (COL3), 13J1.112 (COL2), 13J1.113 (COL1), 13J1.114 (COL0), 13J1.15 (VSS), 13J1.31 (VSS), 13J1.45 (VSS), 13J1.61 (VSS), 13J1.75 (VSS), 13J1.91 (VSS), 13J1.94 (TEST), 16J1.1 (VSS), 16J1.105 (VSS), 16J1.15 (VSS), 16J1.21 (TEST), 16J1.31 (VSS), 16J1.36 (VDE), 16J1.45 (VSS), 16J1.61 (VSS), 16J1.75 (VSS), 16J1.91 (VSS), 16K1.14 (VSS), 16K1.20 (~{CS1}), 16L1.14 (VSS)
- new net ZA1H: 13J1.101 (ZA1H), 16J1.50 (ZA1H)
- new net ZA2H: 13J1.100 (ZA2H), 16J1.51 (ZA2H)
- new net ZA4H: 13J1.99 (ZA4H), 16J1.52 (ZA4H)
- new net ZB1H: 13J1.106 (ZB1H), 16J1.47 (ZB1H)
- new net ZB2H: 13J1.103 (ZB2H), 16J1.48 (ZB2H)
- new net ZB4H: 13J1.102 (ZB4H), 16J1.49 (ZB3H)
- new net ~{BE}: 13J1.98 (~{BE}), 16J1.53 (~{BE})
- new net ~{CSYNC}: 13J1.76 (~{CSYNC})
- new net ~{HBLANK}: 13J1.70 (~{HBLANK})
- new net ~{HSYNC}: 13J1.73 (~{HSYNC})
- new net ~{IRQ}: 16J1.87 (~{IRQ})
- new net ~{RCS1}: 16J1.93 (~{RCS1}), 16L1.20 (~{CS1})
- new net ~{RESET}: 13J1.92 (~{RESET}), 16J1.55 (~{RESET})
- new net ~{ROE1}: 16J1.95 (~{ROE1}), 16L1.22 (~{OE})
- new net ~{ROE2}: 16J1.96 (~{ROE2}), 16K1.22 (~{OE})
- new net ~{RWE1}: 16J1.107 (~{RWE1}), 16L1.27 (~{WE})
- new net ~{RWE2}: 16J1.108 (~{RWE2}), 16K1.27 (~{WE})
- new net ~{SYSRES}: H1.8
- new net ~{UDS}: 16J1.81 (AB13)
- new net ~{VBLANK}: 13J1.69 (~{VBLANK})
- new net ~{VRAM}: 13J1.97 (CR~{CS}), 16J1.54 (CR~{CS}), 16J1.84 (~{VCS})
- new net ~{VSYNC}: 13J1.72 (~{VSYNC})
- no-connect marks 0 -> 27
Other:
- note added: "CRYSTAL OSC 24MHz"
- note added: "SR64KW X 2"
- note added: "VSS"
- note added: "copied over from Sunset Riders Not fully checked yet"
