File: cores/rollerg/sch/Objects.kicad_sch (KiCad schematic)
At the start: 0 parts

Commit message: wip rollerg sch: objects page
Parts:
- added G16: 74LS32, symbol jt74:74LS32
- added G4: MB8464A, Package_SO:SOP-28_8.4x18.16mm_P1.27mm, symbol Memory_RAM:HY6264AxJ
- added G7: 27C1000, symbol jt_rom:27C1000
- added J13: SRAM2K8B, symbol jt_ram:SRAM2K8B
- added J14: 74LS245, symbol jt74:74LS245
- added J3: 053244, symbol konami:053244
- added J9: 053245, symbol konami:053245
- added K2, K8: HN624116P, symbol konami:HN624116P
Connections:
- new net: G16.8, J9.7 (OBJ~{CS})
- new net AR0: J3.30 (AR2), J9.119 (AR0)
- new net AR1: J3.32 (AR1), J9.118 (AR1)
- new net AR2: J3.33 (AR0), J9.117 (AR2)
- new net AROK: J3.34 (AROK), J9.116 (AROK)
- new net BR0: J3.35 (BR2), J9.115 (BR0)
- new net BR1: J3.36 (BR1), J9.114 (BR1)
- new net BR2: J3.37 (BR0), J9.113 (BR2)
- new net BROK: J3.38 (BR0K), J9.112 (BROK)
- new net CLAT: J3.64 (CLAT), J9.86 (CLAT)
- new net CPU~{EN}: J9.26 (CPU)
- new net DB0: J14.2 (A0)
- new net DB1: J14.3 (A1)
- new net DB2: J14.4 (A2)
- new net DB3: J14.5 (A3)
- new net DB4: J14.6 (A4)
- new net DB5: J14.7 (A5)
- new net DB6: J14.8 (A6)
- new net DB7: J14.9 (A7)
- new net HP0: J3.54 (HP0), J9.96 (HP0)
- new net HP1: J3.53 (HP1), J9.97 (HP1)
- new net HP2: J3.52 (HP2), J9.98 (HP2)
- new net HP3: J3.50 (HP3), J9.99 (HP3)
- new net HP4: J3.49 (HP4), J9.100 (HP4)
- new net HP5: J3.48 (HP5), J9.102 (HP5)
- new net HP6: J3.47 (HP6), J9.103 (HP6)
- new net HP7: J3.45 (HP7), J9.104 (HP7)
- new net HP8: J3.44 (HP8), J9.105 (HP8)
- new net HP9: J3.43 (HP9), J9.107 (HP9)
- new net HRFP: J3.39 (HRFP), J9.110 (HRFP)
- new net M12: J3.12 (M12), J9.12 (M12)
- new net M6: J3.10 (M6), J9.10 (M6)
- new net MAIN_A0: G4.10 (A0), G7.12 (A0), J3.19 (AD1), J9.9 (~{LDS})
- new net MAIN_A1: G4.9 (A1), G7.11 (A1), J3.18 (AD2), J9.25 (AD1)
- new net MAIN_A10: G4.21 (A10), G7.23 (A10), J9.14 (AD10)
- new net MAIN_A11: G4.23 (A11), G7.25 (A11)
- new net MAIN_A12: G4.2 (A12), G7.4 (A12)
- new net MAIN_A13: G7.28 (A13)
- new net MAIN_A14: G7.29 (A14)
- new net MAIN_A15: G7.3 (A15)
- new net MAIN_A16: G7.2 (A16)
- new net MAIN_A2: G4.8 (A2), G7.10 (A2), J3.17 (AD3), J9.24 (AD2)
- new net MAIN_A3: G4.7 (A3), G7.9 (A3), J3.15 (AD4), J9.23 (AD3)
- new net MAIN_A4: G4.6 (A4), G7.8 (A4), J9.22 (AD4)
- new net MAIN_A5: G4.5 (A5), G7.7 (A5), J9.20 (AD5)
- new net MAIN_A6: G4.4 (A6), G7.6 (A6), J9.19 (AD6)
- new net MAIN_A7: G4.3 (A7), G7.5 (A7), J9.18 (AD7)
- new net MAIN_A8: G4.25 (A8), G7.27 (A8), J9.17 (AD8)
- new net MAIN_A9: G4.24 (A9), G7.26 (A9), J9.15 (AD9)
- new net MAIN_D0: G4.11 (I/O0), G7.13 (D0), J3.29 (MDB0)
- new net MAIN_D1: G4.12 (I/O1), G7.14 (D1), J3.28 (MDB1)
- new net MAIN_D2: G4.13 (I/O2), G7.15 (D2), J3.27 (MDB2)
- new net MAIN_D3: G4.15 (I/O3), G7.17 (D3), J3.26 (MDB3)
- new net MAIN_D4: G4.16 (I/O4), G7.18 (D4), J3.25 (MDB4)
- new net MAIN_D5: G4.17 (I/O5), G7.19 (D5), J3.24 (MDB5)
- new net MAIN_D6: G4.18 (I/O6), G7.20 (D6), J3.23 (MDB6)
- new net MAIN_D7: G4.19 (I/O7), G7.21 (D7), J3.22 (MDB7)
- new net OBJPXL0: J3.120 (OBO0)
- new net OBJPXL1: J3.119 (OBO1)
- new net OBJPXL2: J3.118 (OBO2)
- new net OBJPXL3: J3.117 (OBO3)
- new net OBJPXL4: J3.116 (OBO4)
- new net OBJPXL5: J3.115 (OBO5)
- new net OBJPXL6: J3.114 (OBO6)
- new net OBJPXL7: J3.113 (OBO7)
- new net OBJPXL8: J3.112 (OBO8)
- new net OBJRAMD0: J13.9 (D0), J14.18 (B0), J9.45 (RD0)
- new net OBJRAMD1: J13.10 (D1), J14.17 (B1), J9.44 (RD1)
- new net OBJRAMD10: J9.33 (RD10)
- new net OBJRAMD11: J9.32 (RD11)
- new net OBJRAMD12: J9.30 (RD12)
- new net OBJRAMD13: J9.29 (RD13)
- new net OBJRAMD14: J9.28 (RD14)
- new net OBJRAMD15: J9.27 (RD15)
- new net OBJRAMD2: J13.11 (D2), J14.16 (B2), J9.43 (RD2)
- new net OBJRAMD3: J13.13 (D3), J14.15 (B3), J9.42 (RD3)
- new net OBJRAMD4: J13.14 (D4), J14.14 (B4), J9.40 (RD4)
- new net OBJRAMD5: J13.15 (D5), J14.13 (B5), J9.39 (RD5)
- new net OBJRAMD6: J13.16 (D6), J14.12 (B6), J9.38 (RD6)
- new net OBJRAMD7: J13.17 (D7), J14.11 (B7), J9.37 (RD7)
- new net OBJRAMD8: J9.35 (RD8)
- new net OBJRAMD9: J9.34 (RD9)
- new net OBJROMA0: J9.85 (CA0), K2.10 (A0), K8.10 (A0)
- new net OBJROMA1: J9.84 (CA1), K2.9 (A1), K8.9 (A1)
- new net OBJROMA10: J9.73 (CA10), K2.39 (A10), K8.39 (A10)
- new net OBJROMA11: J9.72 (CA11), K2.38 (A11), K8.38 (A11)
- new net OBJROMA12: J9.70 (CA12), K2.37 (A12), K8.37 (A12)
- new net OBJROMA13: J9.69 (CA13), K2.36 (A13), K8.36 (A13)
- new net OBJROMA14: J9.68 (CA14), K2.35 (A14), K8.35 (A14)
- new net OBJROMA15: J9.67 (CA15), K2.34 (A15), K8.34 (A15)
- new net OBJROMA16: J9.66 (CA16), K2.33 (A16), K8.33 (A16)
- new net OBJROMA17: J9.65 (CA17), K2.2 (A17), K8.2 (A17)
- new net OBJROMA18: J9.64 (CA18), K2.1 (A18), K8.1 (A18)
- new net OBJROMA2: J9.83 (CA2), K2.8 (A2), K8.8 (A2)
- new net OBJROMA3: J9.82 (CA3), K2.7 (A3), K8.7 (A3)
- new net OBJROMA4: J9.80 (CA4), K2.6 (A4), K8.6 (A4)
- new net OBJROMA5: J9.79 (CA5), K2.5 (A5), K8.5 (A5)
- new net OBJROMA6: J9.78 (CA6), K2.4 (A6), K8.4 (A6)
- new net OBJROMA7: J9.77 (CA7), K2.3 (A7), K8.3 (A7)
- new net OBJROMA8: J9.75 (CA8), K2.41 (A8), K8.41 (A8)
- new net OBJROMA9: J9.74 (CA9), K2.40 (A9), K8.40 (A9)
- new net OBJROMD0: J3.100 (OBJROMD0), K2.14 (D0)
- new net OBJROMD1: J3.99 (OBJROMD1), K2.16 (D1)
- new net OBJROMD10: J3.89 (OBJROMD10), K8.18 (D2)
- new net OBJROMD11: J3.88 (OBJROMD11), K8.20 (D3)
- new net OBJROMD12: J3.87 (OBJROMD12), K8.23 (D4)
- new net OBJROMD13: J3.86 (OBJROMD13), K8.25 (D5)
- new net OBJROMD14: J3.85 (OBJROMD14), K8.27 (D6)
- new net OBJROMD15: J3.84 (OBJROMD15), K8.29 (D7)
- new net OBJROMD16: J3.83 (OBJROMD16), K2.15 (D8)
- new net OBJROMD17: J3.82 (OBJROMD17), K2.17 (D9)
- new net OBJROMD18: J3.80 (OBJROMD18), K2.19 (D10)
- new net OBJROMD19: J3.79 (OBJROMD19), K2.21 (D11)
- new net OBJROMD2: J3.98 (OBJROMD2), K2.18 (D2)
- new net OBJROMD20: J3.78 (OBJROMD20), K2.24 (D12)
- new net OBJROMD21: J3.77 (OBJROMD21), K2.26 (D13)
- new net OBJROMD22: J3.75 (OBJROMD22), K2.28 (D14)
- new net OBJROMD23: J3.74 (OBJROMD23), K2.30 (D15/A-1)
- new net OBJROMD24: J3.73 (OBJROMD24), K8.15 (D8)
- new net OBJROMD25: J3.72 (OBJROMD25), K8.17 (D9)
- new net OBJROMD26: J3.70 (OBJROMD26), K8.19 (D10)
- new net OBJROMD27: J3.69 (OBJROMD27), K8.21 (D11)
- new net OBJROMD28: J3.68 (OBJROMD28), K8.24 (D12)
- new net OBJROMD29: J3.67 (OBJROMD29), K8.26 (D13)
- new net OBJROMD3: J3.97 (OBJROMD3), K2.20 (D3)
- new net OBJROMD30: J3.66 (OBJROMD30), K8.28 (D14)
- new net OBJROMD31: J3.65 (OBJROMD31), K8.30 (D15/A-1)
- new net OBJROMD4: J3.96 (OBJROMD4), K2.23 (D4)
- new net OBJROMD5: J3.95 (OBJROMD5), K2.25 (D5)
- new net OBJROMD6: J3.94 (OBJROMD6), K2.27 (D6)
- new net OBJROMD7: J3.93 (OBJROMD7), K2.29 (D7)
- new net OBJROMD8: J3.92 (OBJROMD8), K8.14 (D0)
- new net OBJROMD9: J3.90 (OBJROMD9), K8.16 (D1)
- new net ORAMA0: J13.1 (A7), J9.50 (RA0)
- new net ORAMA1: J13.4 (A4), J9.52 (RA1)
- new net ORAMA10: J13.2 (A6), J9.63 (RA10)
- new net ORAMA2: J13.5 (A3), J9.53 (RA2)
- new net ORAMA3: J13.23 (A8), J9.54 (RA3)
- new net ORAMA4: J13.6 (A2), J9.55 (RA4)
- new net ORAMA5: J13.22 (A9), J9.56 (RA5)
- new net ORAMA6: J13.7 (A1), J9.57 (RA6)
- new net ORAMA7: J13.8 (A0), J9.58 (RA7)
- new net ORAMA8: J13.19 (A10), J9.59 (RA8)
- new net ORAMA9: J13.3 (A5), J9.62 (RA9)
- new net PL0: J3.63 (PL0), J9.87 (PL0)
- new net PL1: J3.62 (PL1), J9.88 (PL1)
- new net PL2: J3.60 (PL2), J9.89 (PL2)
- new net PL3: J3.59 (PL3), J9.90 (PL3)
- new net PL4: J3.58 (PL4), J9.92 (PL4)
- new net PL5: J3.57 (PL5), J9.93 (PL5)
- new net PL6: J3.56 (PL6), J9.94 (PL6)
- new net PR13: J3.110 (OBO9)
- new net PR14: J3.109 (OBO10)
- new net R/~{W}: G16.9, G4.27 (~{WE})
- new net R~{OE}: J13.20 (~{OE}), J9.49 (R~{OE})
- new net SDI0: J3.108 (OBO11)
- new net SHADOW: J3.55 (SHADOW), J9.95 (SHADOW)
- new net VCC: G4.28 (VCC), G7.1 (VPP), G7.31 (~{PGM}), G7.32 (VCC), J13.24 (VCC), J3.106 (VCC), J3.16 (VCC), J3.46 (VCC), J3.76 (VCC), J9.106 (VCC), J9.120 (VCC), J9.16 (VCC), J9.46 (VCC), J9.60 (VCC), J9.76 (VCC), K2.22 (VCC), K2.32 (BHE), K2.42 (A19), K8.22 (VCC), K8.32 (BHE), K8.42 (A19)
- new net VSS: G4.14 (GND), G7.16 (GND), G7.22 (~{CE}), J13.12 (VSS), J13.18 (~{CS}), J3.1 (VSS), J3.101 (VSS), J3.11 (VSS), J3.111 (VSS), J3.2 (TEST), J3.21 (VSS), J3.31 (VSS), J3.41 (VSS), J3.51 (VSS), J3.61 (VSS), J3.71 (VSS), J3.81 (VSS), J3.91 (VSS), J9.1 (VSS), J9.101 (VSS), J9.11 (VSS), J9.111 (VSS), J9.2 (TEST), J9.21 (VSS), J9.31 (VSS), J9.41 (VSS), J9.51 (VSS), J9.61 (VSS), J9.71 (VSS), J9.8 (~{UDS}), J9.81 (VSS), J9.91 (VSS), K2.11 (~{CE}), K2.12 (VSS), K2.13 (~{OE}), K2.31 (VSS), K8.11 (~{CE}), K8.12 (VSS), K8.13 (~{OE}), K8.31 (VSS)
- new net ~{DS}: J3.14 (~{DS})
- new net ~{HIT}: J3.42 (~{HIT}), J9.108 (~{HIT})
- new net ~{HSYNC}: J3.8 (~{HSYNC}), J9.4 (~{HSYNC})
- new net ~{OBJSET}: J3.13 (OBJ~{SET}), J9.6 (OBJ~{SET})
- new net ~{OBJ_CS}: G16.10
- new net ~{RCS0}: J3.3 (~{RESET}), J9.3 (~{RESET})
- new net ~{RD}: G16.13, G4.22 (~{OE}), J3.20 (~{RD}), J9.13 (~{RD})
- new net ~{VSYNC}: J3.9 (~{VSYNC}), J9.5 (~{VSYNC})
- new net ~{WE1}: J13.21 (~{WR}), J9.48 (~{WE}1)
- new net ~{WE2}: J9.47 (~{WE}2)
- new net ~{ZLD}: J3.40 (~{ZLD}), J9.109 (~{ZLD})
- no-connect marks 0 -> 9
Other:
- note added: "IGUAL"
- note added: "ROM's MASK OF THE SPRITES"
- note added: "VSS"

Commit message: wip rollerg sch: PSAC progress
Connections:
- net M12 renamed M12B
Changed lines of the file:
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@@
 		)
 	)
-	(label "M12"
+	(label "M12B"
 		(at 281.94 187.96 0)
 		(effects
@@
 		)
 	)
-	(hierarchical_label "M12"
+	(hierarchical_label "M12B"
 		(shape input)
 		(at 115.57 104.14 90)

Commit message: wip rollerg sch: PSAC
Parts:
- removed unit 4 of G16
- added F14: 74LS04, symbol jt74:74LS04
Connections:
- net ~{OBJ_CS}: now also F14.10
- net OBOK: now reaches J3.107 (OBOK)
- new net VD6: F14.11
- no-connect marks 9 -> 8
Other:
- note removed: "IGUAL"
Changed lines of the file:
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@@
 	)
 	(no_connect
-		(at 386.08 157.48)
-	)
-	(no_connect
 		(at 292.1 134.62)
 	)
@@
 	(wire
 		(pts
+			(xy 33.02 133.35) (xy 36.83 133.35)
+		)
+		(stroke
+			(width 0)
+			(type default)
+		)
+	)
+	(wire
+		(pts
 			(xy 196.85 151.13) (xy 208.28 151.13)
 		)
@@
 		)
 	)
+	(wire
+		(pts
+			(xy 391.16 157.48) (xy 386.08 157.48)
+		)
+		(stroke
+			(width 0)
+			(type default)
+		)
+	)
 	(bus
 		(pts
@@
 	(wire
 		(pts
+			(xy 52.07 133.35) (xy 66.04 133.35)
+		)
+		(stroke
+			(width 0)
+			(type default)
+		)
+	)
+	(wire
+		(pts
 			(xy 213.36 110.49) (xy 229.87 110.49)
 		)
@@
 		)
 	)
-	(rectangle
-		(start 106.68 201.93)
-		(end 392.43 218.44)
-		(stroke
-			(width 0.254)
-			(type default)
-		)
-		(fill
-			(type none)
-		)
-	)
-	(rectangle
-		(start 295.91 218.44)
-		(end 330.2 229.87)
-		(stroke
-			(width 0.254)
-			(type default)
-		)
-		(fill
-			(type none)
-		)
-	)
 	(image
 		(at 396.24 260.35)
@@
 		)
 	)
-	(text "IGUAL"
-		(exclude_from_sim no)
-		(at 312.674 224.536 0)
-		(effects
-			(font
-				(size 3.81 3.81)
-			)
-		)
-	)
 	(text "VSS"
 		(exclude_from_sim no)
@@
 		)
 	)
+	(label "~{OBJ_CS}"
+		(at 62.23 133.35 180)
+		(effects
+			(font
+				(size 1.27 1.27)
+			)
+			(justify right bottom)
+		)
+	)
 	(label "OBJROMA16"
 		(at 161.29 96.52 270)
@@
 		)
 	)
-	(hierarchical_label "~{OBJ_CS}"
-		(shape input)
-		(at 66.04 133.35 180)
-		(effects
-			(font
-				(size 1.27 1.27)
-			)
-			(justify right)
-		)
-	)
 	(hierarchical_label "MAIN_D[15..0]"
 		(shape tri_state)
@@
 		)
 	)
+	(hierarchical_label "VD6"
+		(shape input)
+		(at 33.02 133.35 180)
+		(effects
+			(font
+				(size 1.27 1.27)
+			)
+			(justify right)
+		)
+	)
 	(hierarchical_label "PR13"
 		(shape output)
@@
 		)
 	)
-	(hierarchical_label "DB[7..0]"
-		(shape tri_state)
-		(at 219.71 196.85 180)
+	(hierarchical_label "OBOK"
+		(shape output)
+		(at 391.16 157.48 0)
 		(effects
 			(font
 				(size 1.27 1.27)
 			)
-			(justify right)
+			(justify left)
 		)
 	)
-	(hierarchical_label "~{RD}"
-		(shape input)
-		(at 29.21 101.6 180)
+	(hierarchical_label "DB[7..0]"
+		(shape tri_state)
+		(at 219.71 196.85 180)
 		(effects
 			(font
@@
 	)
 	(symbol
-		(lib_name "74LS32_1")
-		(lib_id "jt74:74LS32")
-		(at 36.83 99.06 0)
-		(unit 4)
+		(lib_id "jt74:74LS04")
+		(at 44.45 133.35 0)
+		(unit 5)
 		(exclude_from_sim no)
 		(in_bom yes)
@@
 		(dnp no)
 		(fields_autoplaced yes)
-		(property "Reference" "G16"
-			(at 36.83 90.17 0)
+		(property "Reference" "F14"
+			(at 44.45 124.46 0)
 			(effects
 				(font
@@
 			)
 		)
-		(property "Value" "74LS32"
-			(at 36.83 92.71 0)
+		(property "Value" "74LS04"
+			(at 44.45 127 0)
 			(effects
 				(font
@@
 		)
 		(property "Footprint" ""
-			(at 36.83 99.06 0)
+			(at 44.45 133.35 0)
 			(effects
 				(font
@@
 			)
 		)
-		(property "Datasheet" "http://www.ti.com/lit/gpn/sn74LS32"
-			(at 36.83 99.06 0)
+		(property "Datasheet" "http://www.ti.com/lit/gpn/sn74LS04"
+			(at 44.45 133.35 0)
 			(effects
 				(font
@@
 			)
 		)
-		(property "Description" "Quad 2-input OR"
-			(at 36.83 99.06 0)
+		(property "Description" "Hex Inverter"
+			(at 44.45 133.35 0)
 			(effects
 				(font
@@
 			)
 		)
-		(pin "10"
-		)
-		(pin "14"
+		(pin "6"
 		)
-		(pin "4"
+		(pin "9"
 		)
-		(pin "13"
+		(pin "7"
 		)
-		(pin "6"
+		(pin "8"
 		)
-		(pin "12"
+		(pin "2"
 		)
 		(pin "3"
 		)
-		(pin "9"
+		(pin "4"
 		)
-		(pin "7"
+		(pin "11"
 		)
-		(pin "2"
+		(pin "10"
+		)
+		(pin "12"
+		)
+		(pin "13"
 		)
 		(pin "5"
@@
 		(pin "1"
 		)
-		(pin "11"
-		)
-		(pin "8"
+		(pin "14"
 		)
 		(instances
-			(project ""
+			(project "rollerg"
 				(path "/bb61a05c-9ea0-4d47-a326-1f7e835840f3/352c0ec6-92f1-4542-b6d5-7e0d5161301b"
-					(reference "G16")
-					(unit 4)
+					(reference "F14")
+					(unit 5)
 				)
 			)

Commit message: wip rollerg sch: SOUND
Parts:
- added unit 3 of F14
- added F16: 74LS08, symbol 74xx:74LS08
- added unit 1 of G16
- added unit 4 of G16
Connections:
- net CPU~{EN}: now also G16.2
- net DB0: now also J3.29 (MDB0)
- net DB1: now also J3.28 (MDB1)
- net DB2: now also J3.27 (MDB2)
- net DB3: now also J3.26 (MDB3)
- net DB4: now also J3.25 (MDB4)
- net DB5: now also J3.24 (MDB5)
- net DB6: now also J3.23 (MDB6)
- net DB7: now also J3.22 (MDB7)
- net MAIN_D0: no longer J3.29 (MDB0)
- net MAIN_D1: no longer J3.28 (MDB1)
- net MAIN_D2: no longer J3.27 (MDB2)
- net MAIN_D3: no longer J3.26 (MDB3)
- net MAIN_D4: no longer J3.25 (MDB4)
- net MAIN_D5: no longer J3.24 (MDB5)
- net MAIN_D6: no longer J3.23 (MDB6)
- net MAIN_D7: no longer J3.22 (MDB7)
- net VCC: now also G4.26 (CS2)
- net ~{OBJ_CS}: now also F16.10
- net ~{RD}: now also G16.13
- net at J14.1 (A->B): now also G16.11
- net at J14.19 (~{CE}): now also G16.3
- net ~{CS1}: now reaches G4.20 (~{CS1})
- net OOE: now reaches G7.24 (~{OE})
- net M6 renamed CLK2
- net MAIN_A13 renamed MAIN_AB0
- net MAIN_A14 renamed MAIN_AB1
- net MAIN_A15 renamed MAIN_AB2
- net MAIN_A16 renamed MAIN_AB3
- new net: F16.8, G16.1
- new net: F14.6, G16.12
- new net PAL15: F14.5, F16.9

Commit message: almost complete rollerg sch
Connections:
- net PAL15 is gone; now on net ~{OBJSET}: F14.5, F16.9
- net OBJPXL8 renamed OBOB
- net OBJRAMD10: no longer names the net of J9.33 (RD10)
- net OBJRAMD11: no longer names the net of J9.32 (RD11)
- net OBJRAMD12: no longer names the net of J9.30 (RD12)
- net OBJRAMD13: no longer names the net of J9.29 (RD13)
- net OBJRAMD14: no longer names the net of J9.28 (RD14)
- net OBJRAMD15: no longer names the net of J9.27 (RD15)
- net OBJRAMD8: no longer names the net of J9.35 (RD8)
- net OBJRAMD9: no longer names the net of J9.34 (RD9)
- net PR13: no longer names the net of J3.110 (OBO9)
- net PR14: no longer names the net of J3.109 (OBO10)
- net ~{RCS0} renamed RES
- net ~{WE2}: no longer names the net of J9.47 (~{WE}2)
- no-connect marks 8 -> 19
