File: cores/rollerg/sch/RGB.kicad_sch (KiCad schematic)
At the start: 22 parts

Commit message: almost complete rollerg sch
Parts:
- removed unit 2 of D18
- removed unit 4 of D18
- removed F7: 74LS04, symbol jt74:74LS04
- added unit 4 of D18
Connections:
- net CA19 is gone; now on net MAIN_A0: F7.13
- net ~{DS}: now also D18.13
- net ~{HBK}: now also H24.1 (A)
- net ~{VBK}: now also H24.2 (B)
- net OBCE: now reaches E18.19 (~{CE})
- net COLABR4: now reaches C14.13 (D4)
- net COLABR4: now also E15.14 (D4), E16.14 (B4)
- net COLABR5: now reaches C14.14 (D5)
- net COLABR5: now also E15.15 (D5), E16.13 (B5)
- net COLABR6: now reaches C14.17 (D6)
- net COLABR6: now also E15.16 (D6), E16.12 (B6)
- net COLABR7: now reaches C14.18 (D7)
- net COLABR7: now also E15.17 (D7), E16.11 (B7)
- net COLABR0: now reaches C14.3 (D0)
- net COLABR0: now also E15.9 (D0), E16.18 (B0)
- net COLABR1: now reaches C14.4 (D1)
- net COLABR1: now also E15.10 (D1), E16.17 (B1)
- net COLABR2: now reaches C14.7 (D2)
- net COLABR2: now also E15.11 (D2), E16.16 (B2)
- net COLABR3: now reaches C14.8 (D3)
- net COLABR3: now also E15.13 (D3), E16.15 (B3)
- net at D18.3, E16.19 (~{CE}): now also D18.12
- net at E15.21 (~{WR}): now also D18.11
- net VSS renamed GNDPWR
- no-connect marks 3 -> 12
Other:
- moved on the sheet: D18A, F7F
