File: cores/rollerg/sch/Not_Populated.kicad_sch (KiCad schematic)
At the start: 0 parts

Commit message: almost complete rollerg sch
Parts:
- added C11, C7: 23C4100, symbol jt_rom:23C4100
- added CN1, CN2, CN3, CN4: Conn_02x32_Row_Letter_First, symbol Connector_Generic:Conn_02x32_Row_Letter_First

Commit message: half unpopulated sheet
Parts:
- removed C7: 23C4100, symbol jt_rom:23C4100
- added K13, K19: 23C4100, symbol jt_rom:23C4100
- added U2, U3, U6, U7: 74LS244, symbol 74xx:74LS244
Connections:
- net VCC: now reaches CN3.a1 (Pin_a1)
- net VCC: now also CN2.a1 (Pin_a1), CN2.a2 (Pin_a2), CN2.a3 (Pin_a3), CN2.a4 (Pin_a4), CN2.a5 (Pin_a5), CN2.b1 (Pin_b1), CN2.b2 (Pin_b2), CN2.b3 (Pin_b3), CN2.b4 (Pin_b4), CN2.b5 (Pin_b5), CN3.a2 (Pin_a2), CN3.b1 (Pin_b1), CN3.b2 (Pin_b2), K13.21 (VCC), K13.31 (~{BYTE}), K19.21 (VCC), K19.31 (~{BYTE})
- net OBJROMA6: now reaches CN3.a10 (Pin_a10)
- net OBJROMA6: now also K13.3 (A6), K19.3 (A6)
- net OBJROMA7: now reaches CN3.a11 (Pin_a11)
- net OBJROMA7: now also K13.2 (A7), K19.2 (A7)
- net OBJROMA8: now reaches CN3.a12 (Pin_a12)
- net OBJROMA8: now also K13.40 (A8), K19.40 (A8)
- net OBJROMA9: now reaches CN3.a13 (Pin_a13)
- net OBJROMA9: now also K13.39 (A9), K19.39 (A9)
- net at CN3.a14 (Pin_a14): now also U6.2 (I0a)
- net at CN3.a15 (Pin_a15): now also U6.4 (I1a)
- net at CN3.a16 (Pin_a16): now also U6.6 (I2a)
- net at CN3.a17 (Pin_a17): now also U6.8 (I3a)
- net at CN3.a18 (Pin_a18): now also U6.17 (I3b)
- net at CN3.a19 (Pin_a19): now also U6.15 (I2b)
- net at CN3.a20 (Pin_a20): now also U6.13 (I1b)
- net at CN3.a21 (Pin_a21): now also U6.11 (I0b)
- net at CN3.a22 (Pin_a22): now also U7.2 (I0a)
- net at CN3.a23 (Pin_a23): now also U7.4 (I1a)
- net at CN3.a24 (Pin_a24): now also U7.6 (I2a)
- net at CN3.a25 (Pin_a25): now also U7.8 (I3a)
- net at CN3.a26 (Pin_a26): now also U7.17 (I3b)
- net at CN3.a27 (Pin_a27): now also U7.15 (I2b)
- net at CN3.a28 (Pin_a28): now also U7.13 (I1b)
- net at CN3.a29 (Pin_a29): now also U7.11 (I0b)
- net VSS: now reaches CN3.a30 (Pin_a30)
- net VSS: now also CN1.b12 (Pin_b12), CN2.a28 (Pin_a28), CN2.a29 (Pin_a29), CN2.a30 (Pin_a30), CN2.a31 (Pin_a31), CN2.a32 (Pin_a32), CN2.b28 (Pin_b28), CN2.b29 (Pin_b29), CN2.b30 (Pin_b30), CN2.b31 (Pin_b31), CN2.b32 (Pin_b32), CN3.a31 (Pin_a31), CN3.a32 (Pin_a32), CN3.b12 (Pin_b12), CN3.b13 (Pin_b13), CN3.b30 (Pin_b30), CN3.b31 (Pin_b31), CN3.b32 (Pin_b32), K13.10 (~{CE}), K13.11 (VSS), K13.30 (VSS), K19.10 (~{CE}), K19.11 (VSS), K19.30 (VSS)
- net OBJROMA0: now reaches CN3.a4 (Pin_a4)
- net OBJROMA0: now also K13.9 (A0), K19.9 (A0)
- net OBJROMA1: now reaches CN3.a5 (Pin_a5)
- net OBJROMA1: now also K13.8 (A1), K19.8 (A1)
- net OBJROMA2: now reaches CN3.a6 (Pin_a6)
- net OBJROMA2: now also K13.7 (A2), K19.7 (A2)
- net OBJROMA3: now reaches CN3.a7 (Pin_a7)
- net OBJROMA3: now also K13.6 (A3), K19.6 (A3)
- net OBJROMA4: now reaches CN3.a8 (Pin_a8)
- net OBJROMA4: now also K13.5 (A4), K19.5 (A4)
- net OBJROMA5: now reaches CN3.a9 (Pin_a9)
- net OBJROMA5: now also K13.4 (A5), K19.4 (A5)
- net OBJROMA16: now reaches CN3.b10 (Pin_b10)
- net OBJROMA16: now also K13.32 (A16), K19.32 (A16)
- net OBJROMA17: now reaches CN3.b11 (Pin_b11)
- net OBJROMA17: now also K13.1 (A17), K19.1 (A17)
- net at CN3.b14 (Pin_b14): now also U2.2 (I0a)
- net at CN3.b15 (Pin_b15): now also U2.4 (I1a)
- net at CN3.b16 (Pin_b16): now also U2.6 (I2a)
- net at CN3.b17 (Pin_b17): now also U2.8 (I3a)
- net at CN3.b18 (Pin_b18): now also U2.17 (I3b)
- net at CN3.b19 (Pin_b19): now also U2.15 (I2b)
- net at CN3.b20 (Pin_b20): now also U2.13 (I1b)
- net at CN3.b21 (Pin_b21): now also U2.11 (I0b)
- net at CN3.b22 (Pin_b22): now also U3.2 (I0a)
- net at CN3.b23 (Pin_b23): now also U3.4 (I1a)
- net at CN3.b24 (Pin_b24): now also U3.6 (I2a)
- net at CN3.b25 (Pin_b25): now also U3.8 (I3a)
- net at CN3.b26 (Pin_b26): now also U3.17 (I3b)
- net at CN3.b27 (Pin_b27): now also U3.15 (I2b)
- net at CN3.b28 (Pin_b28): now also U3.13 (I1b)
- net at CN3.b29 (Pin_b29): now also U3.11 (I0b)
- net OBJROMA10: now reaches CN3.b4 (Pin_b4)
- net OBJROMA10: now also K13.38 (A10), K19.38 (A10)
- net OBJROMA11: now reaches CN3.b5 (Pin_b5)
- net OBJROMA11: now also K13.37 (A11), K19.37 (A11)
- net OBJROMA12: now reaches CN3.b6 (Pin_b6)
- net OBJROMA12: now also K13.36 (A12), K19.36 (A12)
- net OBJROMA13: now reaches CN3.b7 (Pin_b7)
- net OBJROMA13: now also K13.35 (A13), K19.35 (A13)
- net OBJROMA14: now reaches CN3.b8 (Pin_b8)
- net OBJROMA14: now also K13.34 (A14), K19.34 (A14)
- net OBJROMA15: now reaches CN3.b9 (Pin_b9)
- net OBJROMA15: now also K13.33 (A15), K19.33 (A15)
- new net OBJROMD0: K13.13 (D0), U6.18 (O0a)
- new net OBJROMD1: K13.15 (D1), U6.16 (O1a)
- new net OBJROMD10: K19.17 (D2), U2.14 (O2a)
- new net OBJROMD11: K19.19 (D3), U2.12 (O3a)
- new net OBJROMD12: K19.22 (D4), U2.3 (O3b)
- new net OBJROMD13: K19.24 (D5), U2.5 (O2b)
- new net OBJROMD14: K19.26 (D6), U2.7 (O1b)
- new net OBJROMD15: K19.28 (D7), U2.9 (O0b)
- new net OBJROMD16: K13.14 (D8), U7.18 (O0a)
- new net OBJROMD17: K13.16 (D9), U7.16 (O1a)
- new net OBJROMD18: K13.18 (D10), U7.14 (O2a)
- new net OBJROMD19: K13.20 (D11), U7.12 (O3a)
- new net OBJROMD2: K13.17 (D2), U6.14 (O2a)
- new net OBJROMD20: K13.23 (D12), U3.3 (O3b), U7.3 (O3b)
- new net OBJROMD21: K13.25 (D13), U3.5 (O2b), U7.5 (O2b)
- new net OBJROMD22: K13.27 (D14), U3.7 (O1b), U7.7 (O1b)
- new net OBJROMD23: K13.29 ( D15 /A-1), U3.9 (O0b), U7.9 (O0b)
- new net OBJROMD24: K19.14 (D8), U3.18 (O0a)
- new net OBJROMD25: K19.16 (D9), U3.16 (O1a)
- new net OBJROMD26: K19.18 (D10), U3.14 (O2a)
- new net OBJROMD27: K19.20 (D11), U3.12 (O3a)
- new net OBJROMD28: K19.23 (D12)
- new net OBJROMD29: K19.25 (D13)
- new net OBJROMD3: K13.19 (D3), U6.12 (O3a)
- new net OBJROMD30: K19.27 (D14)
- new net OBJROMD31: K19.29 ( D15 /A-1)
- new net OBJROMD4: K13.22 (D4), U6.3 (O3b)
- new net OBJROMD5: K13.24 (D5), U6.5 (O2b)
- new net OBJROMD6: K13.26 (D6), U6.7 (O1b)
- new net OBJROMD7: K13.28 (D7), U6.9 (O0b)
- new net OBJROMD8: K19.13 (D0), U2.18 (O0a)
- new net OBJROMD9: K19.15 (D1), U2.16 (O1a)
- no-connect marks 0 -> 2
Other:
- note added: "There's nothing indicated on the board; my guess is that where a 20-pin connector should go, there will be an LS244 or LS245."
- moved on the sheet: CN3

Commit message: unpopulated sheet
Parts:
- removed C11: 23C4100, symbol jt_rom:23C4100
- removed CN4: Conn_02x32_Row_Letter_First, symbol Connector_Generic:Conn_02x32_Row_Letter_First
- added J2, J4: Conn_02x25_Counter_Clockwise, symbol Connector_Generic:Conn_02x25_Counter_Clockwise
- CN1, CN2, CN3, U2, U3, U6, U7: now not fitted
Connections:
- net VCC: now also CN1.a1 (Pin_a1), CN1.a16 (Pin_a16), CN1.a17 (Pin_a17), CN1.a18 (Pin_a18), CN1.a19 (Pin_a19), CN1.a2 (Pin_a2), CN1.a28 (Pin_a28), CN1.a29 (Pin_a29), CN1.a3 (Pin_a3), CN1.a30 (Pin_a30), CN1.a31 (Pin_a31), CN1.a32 (Pin_a32), CN1.a4 (Pin_a4), CN1.a5 (Pin_a5), CN1.b1 (Pin_b1), CN1.b16 (Pin_b16), CN1.b17 (Pin_b17), CN1.b18 (Pin_b18), CN1.b2 (Pin_b2), CN1.b28 (Pin_b28), CN1.b29 (Pin_b29), CN1.b3 (Pin_b3), CN1.b30 (Pin_b30), CN1.b31 (Pin_b31), CN1.b32 (Pin_b32), CN1.b4 (Pin_b4), CN1.b5 (Pin_b5), CN2.a16 (Pin_a16), CN2.a17 (Pin_a17), CN2.a18 (Pin_a18), CN2.a19 (Pin_a19), CN2.b17 (Pin_b17), CN2.b18 (Pin_b18), CN2.b19 (Pin_b19), J2.38 (Pin_38), J2.50 (Pin_50), J4.12 (Pin_12)
- net VSS: now also CN1.a20 (Pin_a20), CN1.a21 (Pin_a21), CN1.a22 (Pin_a22), CN1.a23 (Pin_a23), CN1.b20 (Pin_b20), CN1.b21 (Pin_b21), CN1.b22 (Pin_b22), CN1.b23 (Pin_b23), CN2.a20 (Pin_a20), CN2.a21 (Pin_a21), CN2.a22 (Pin_a22), CN2.a23 (Pin_a23), CN2.b20 (Pin_b20), CN2.b21 (Pin_b21), CN2.b22 (Pin_b22), CN2.b23 (Pin_b23), J2.1 (Pin_1), J2.10 (Pin_10), J2.11 (Pin_11), J2.12 (Pin_12), J2.13 (Pin_13), J2.14 (Pin_14), J2.15 (Pin_15), J2.16 (Pin_16), J2.17 (Pin_17), J2.18 (Pin_18), J2.19 (Pin_19), J2.2 (Pin_2), J2.20 (Pin_20), J2.21 (Pin_21), J2.22 (Pin_22), J2.23 (Pin_23), J2.24 (Pin_24), J2.25 (Pin_25), J2.3 (Pin_3), J2.4 (Pin_4), J2.5 (Pin_5), J2.6 (Pin_6), J2.7 (Pin_7), J2.8 (Pin_8), J2.9 (Pin_9), J4.26 (Pin_26), J4.27 (Pin_27), J4.28 (Pin_28), J4.29 (Pin_29), J4.30 (Pin_30), J4.31 (Pin_31), J4.32 (Pin_32), J4.33 (Pin_33), J4.34 (Pin_34), J4.35 (Pin_35), J4.36 (Pin_36), J4.37 (Pin_37), J4.38 (Pin_38), J4.39 (Pin_39), J4.40 (Pin_40), J4.41 (Pin_41), J4.42 (Pin_42), J4.43 (Pin_43), J4.44 (Pin_44), J4.45 (Pin_45), J4.46 (Pin_46), J4.47 (Pin_47), J4.48 (Pin_48), J4.49 (Pin_49), J4.50 (Pin_50); no longer CN1.b12 (Pin_b12)
- net RA4: now reaches CN1.a10 (Pin_a10)
- net RA5: now reaches CN1.a11 (Pin_a11)
- net RA6: now reaches CN1.a12 (Pin_a12)
- net RA7: now reaches CN1.a13 (Pin_a13)
- net RA8: now reaches CN1.a14 (Pin_a14)
- net RA9: now reaches CN1.a15 (Pin_a15)
- net RD0: now reaches CN1.a24 (Pin_a24)
- net RD1: now reaches CN1.a25 (Pin_a25)
- net RD2: now reaches CN1.a26 (Pin_a26)
- net RD3: now reaches CN1.a27 (Pin_a27)
- net RA1: now reaches CN1.a7 (Pin_a7)
- net RA2: now reaches CN1.a8 (Pin_a8)
- net RA3: now reaches CN1.a9 (Pin_a9)
- net RA14: now reaches CN1.b10 (Pin_b10)
- net RA15: now reaches CN1.b11 (Pin_b11)
- net RA17: now reaches CN1.b13 (Pin_b13)
- net RA18: now reaches CN1.b14 (Pin_b14)
- net RD4: now reaches CN1.b24 (Pin_b24)
- net RD5: now reaches CN1.b25 (Pin_b25)
- net RD6: now reaches CN1.b26 (Pin_b26)
- net RD7: now reaches CN1.b27 (Pin_b27)
- net RA10: now reaches CN1.b6 (Pin_b6)
- net RA11: now reaches CN1.b7 (Pin_b7)
- net RA12: now reaches CN1.b8 (Pin_b8)
- net RA13: now reaches CN1.b9 (Pin_b9)
- net CA5: now reaches CN2.a10 (Pin_a10)
- net CA6: now reaches CN2.a11 (Pin_a11)
- net CA7: now reaches CN2.a12 (Pin_a12)
- net CA8: now reaches CN2.a13 (Pin_a13)
- net CA9: now reaches CN2.a14 (Pin_a14)
- net CA10: now reaches CN2.a15 (Pin_a15)
- net PRAM0: now reaches CN2.a24 (Pin_a24)
- net PRAM1: now reaches CN2.a25 (Pin_a25)
- net PRAM2: now reaches CN2.a26 (Pin_a26)
- net PRAM3: now reaches CN2.a27 (Pin_a27)
- net CA1: now reaches CN2.a6 (Pin_a6)
- net CA2: now reaches CN2.a7 (Pin_a7)
- net CA3: now reaches CN2.a8 (Pin_a8)
- net CA4: now reaches CN2.a9 (Pin_a9)
- net CA15: now reaches CN2.b10 (Pin_b10)
- net CA16: now reaches CN2.b11 (Pin_b11)
- net CA17: now reaches CN2.b12 (Pin_b12)
- net CA18: now reaches CN2.b13 (Pin_b13)
- net CA19: now reaches CN2.b14 (Pin_b14)
- net PRAM4: now reaches CN2.b24 (Pin_b24)
- net PRAM5: now reaches CN2.b25 (Pin_b25)
- net PRAM6: now reaches CN2.b26 (Pin_b26)
- net PRAM7: now reaches CN2.b27 (Pin_b27)
- net CA11: now reaches CN2.b6 (Pin_b6)
- net CA12: now reaches CN2.b7 (Pin_b7)
- net CA13: now reaches CN2.b8 (Pin_b8)
- net CA14: now reaches CN2.b9 (Pin_b9)
- new net DTAC: J2.32 (Pin_32)
- new net MAIN_A0: J2.28 (Pin_28)
- new net MAIN_A1: J2.29 (Pin_29)
- new net MAIN_A10: J4.13 (Pin_13)
- new net MAIN_A11: J4.14 (Pin_14)
- new net MAIN_A12: J4.11 (Pin_11)
- new net MAIN_A13: J4.10 (Pin_10)
- new net MAIN_A14: J4.9 (Pin_9)
- new net MAIN_A15: J4.8 (Pin_8)
- new net MAIN_A16: J4.6 (Pin_6)
- new net MAIN_A17: J4.7 (Pin_7)
- new net MAIN_A18: J4.4 (Pin_4)
- new net MAIN_A19: J4.5 (Pin_5)
- new net MAIN_A2: J2.26 (Pin_26)
- new net MAIN_A20: J2.46 (Pin_46)
- new net MAIN_A21: J2.45 (Pin_45)
- new net MAIN_A22: J2.44 (Pin_44)
- new net MAIN_A23: J2.43 (Pin_43)
- new net MAIN_A3: J2.27 (Pin_27)
- new net MAIN_A4: J4.25 (Pin_25)
- new net MAIN_A5: J4.24 (Pin_24)
- new net MAIN_A6: J4.23 (Pin_23)
- new net MAIN_A7: J4.22 (Pin_22)
- new net MAIN_A8: J4.15 (Pin_15)
- new net MAIN_A9: J4.16 (Pin_16)
- new net MAIN_D0: J2.41 (Pin_41)
- new net MAIN_D1: J2.40 (Pin_40), J2.42 (Pin_42)
- new net MAIN_D2: J2.39 (Pin_39)
- new net MAIN_D4: J2.37 (Pin_37)
- new net MAIN_D5: J2.36 (Pin_36)
- new net MAIN_D6: J2.35 (Pin_35)
- new net MAIN_D7: J2.34 (Pin_34)
- new net MPE: J2.48 (Pin_48)
- new net MPQ: J2.47 (Pin_47)
- new net RA16: CN1.b12 (Pin_b12)
- new net RESET: J4.21 (Pin_21)
- new net R/~{W}: J2.30 (Pin_30)
- new net ~{AS}: J2.31 (Pin_31)
- new net ~{CLK2}: J2.33 (Pin_33)
- new net ~{DS}: J2.49 (Pin_49)
- new net ~{FIRQ}: J4.18 (Pin_18)
- new net ~{HALT}: J4.20 (Pin_20)
- new net ~{IRQ}: J4.17 (Pin_17)
- new net ~{NMI}: J4.19 (Pin_19)
- no-connect marks 2 -> 9
Other:
- moved on the sheet: K13, K19
