File: cores/rollerg/sch/PSAC.kicad_sch (KiCad schematic)
At the start: 0 parts

Commit message: wip rollerg sch: objects page
Parts:
- added D23, F23: 23C4000, symbol jt_rom:23C4000
- added G16: 74LS32, symbol jt74:74LS32
- added H18: 74LS74, symbol jt74:74LS74
- added H20: 74LS273, symbol 74xx:74LS273
- added H21: 74LS399, symbol 74xx:74LS399
- added I19: 74LS244, symbol 74xx:74LS244
- added I21, J21: 74LS174, symbol 74xx:74LS174
- added I24: ~, symbol konami:051316
- added J16: 74LS04, symbol jt74:74LS04
- added J20: 74LS175, symbol 74xx:74LS175
Connections:
- new net: G16.6, J20.13 (D3)
- new net: H20.13 (D4), J20.2 (Q0)
- new net: H20.14 (D5), J20.7 (Q1)
- new net: H20.3 (D0), H21.2 (Qa)
- new net: H20.4 (D1), H21.7 (Qb)
- new net: H20.7 (D2), H21.10 (Qc)
- new net: H20.8 (D3), H21.15 (Qd)
- new net: H18.11 (C), J20.9 (Cp)
- new net: H21.1 (S), J16.6
- new net CA0: I24.31 (CA0), J16.5
- new net CA1: D23.12 (A0), F23.12 (A0), I24.30 (CA1)
- new net CA10: D23.26 (A9), F23.26 (A9), I24.21 (CA10)
- new net CA11: D23.23 (A10), F23.23 (A10), I24.20 (CA11)
- new net CA12: D23.25 (A11), F23.25 (A11), I24.19 (CA12)
- new net CA13: D23.4 (A12), F23.4 (A12), I24.18 (CA13)
- new net CA14: D23.28 (A13), F23.28 (A13), I24.17 (CA14)
- new net CA15: D23.29 (A14), F23.29 (A14), I24.15 (CA15)
- new net CA16: D23.3 (A15), F23.3 (A15), I24.14 (CA16)
- new net CA17: D23.2 (A16), F23.2 (A16), I24.13 (CA17)
- new net CA18: D23.30 (A17), F23.30 (A17), I24.12 (CA18)
- new net CA2: D23.11 (A1), F23.11 (A1), I24.29 (CA2)
- new net CA3: D23.10 (A2), F23.10 (A2), I24.28 (CA3)
- new net CA4: D23.9 (A3), F23.9 (A3), I24.27 (CA4)
- new net CA5: D23.8 (A4), F23.8 (A4), I24.26 (CA5)
- new net CA6: D23.7 (A5), F23.7 (A5), I24.25 (CA6)
- new net CA7: D23.6 (A6), F23.6 (A6), I24.24 (CA7)
- new net CA8: D23.5 (A7), F23.5 (A7), I24.23 (CA8)
- new net CA9: D23.27 (A8), F23.27 (A8), I24.22 (CA9)
- new net DB0: I19.18 (O0a), I24.50 (DB0)
- new net DB1: I19.16 (O1a), I24.51 (DB1)
- new net DB2: I19.14 (O2a), I24.52 (DB2)
- new net DB3: I19.12 (O3a), I24.53 (DB3)
- new net DB4: I19.9 (O0b), I24.54 (DB4)
- new net DB5: I19.7 (O1b), I24.55 (DB5)
- new net DB6: I19.5 (O2b), I24.56 (DB6)
- new net DB7: I19.3 (O3b), I24.57 (DB7)
- new net G18P15: G16.4
- new net MAIN_A0: J21.3 (D0)
- new net MAIN_A1: J21.4 (D1)
- new net MAIN_A10: I21.13 (D4)
- new net MAIN_A2: J21.6 (D2)
- new net MAIN_A3: J21.11 (D3)
- new net MAIN_A4: J21.13 (D4)
- new net MAIN_A5: J21.14 (D5)
- new net MAIN_A6: I21.3 (D0)
- new net MAIN_A7: I21.4 (D1)
- new net MAIN_A8: I21.6 (D2)
- new net MAIN_A9: I21.11 (D3)
- new net OBLK: G16.5, I24.4 (OBLK)
- new net PA0: I24.36 (A0), J21.2 (Q0)
- new net PA1: I24.37 (A1), J21.5 (Q1)
- new net PA10: I21.12 (Q4), I24.46 (A10)
- new net PA2: I24.38 (A2), J21.7 (Q2)
- new net PA3: I24.39 (A3), J21.10 (Q3)
- new net PA4: I24.40 (A4), J21.12 (Q4)
- new net PA5: I24.41 (A5), J21.15 (Q5)
- new net PA6: I21.2 (Q0), I24.42 (A6)
- new net PA7: I21.5 (Q1), I24.43 (A7)
- new net PA8: I21.7 (Q2), I24.44 (A8)
- new net PA9: I21.10 (Q3), I24.45 (A9)
- new net PRAM0: D23.13 (D0), F23.13 (D0), H21.3 (I0a), I19.2 (I0a)
- new net PRAM1: D23.14 (D1), F23.14 (D1), H21.6 (I0b), I19.4 (I1a)
- new net PRAM2: D23.15 (D2), F23.15 (D2), H21.11 (I0c), I19.6 (I2a)
- new net PRAM3: D23.17 (D3), F23.17 (D3), H21.14 (I0d), I19.8 (I3a)
- new net PRAM4: D23.18 (D4), F23.18 (D4), H21.4 (I1a), I19.11 (I0b)
- new net PRAM5: D23.19 (D5), F23.19 (D5), H21.5 (I1b), I19.13 (I1b)
- new net PRAM6: D23.20 (D6), F23.20 (D6), H21.12 (I1c), I19.15 (I2b)
- new net PRAM7: D23.21 (D7), F23.21 (D7), H21.13 (I1d), I19.17 (I3b)
- new net R/~{W}: I24.58 (RW)
- new net VCC: D23.32 (VCC), F23.32 (VCC)
- new net VSS: D23.16 (GND), F23.16 (GND), I24.16 (GND), I24.3 (GND), I24.35 (GND), I24.48 (GND)
- no-connect marks 0 -> 6

Commit message: wip rollerg sch: PSAC progress
Parts:
- added E14: SRAM2K8B, symbol jt_ram:SRAM2K8B
- added E18: 74LS245, symbol jt74:74LS245
- added E20: 63S141, symbol arcade:N82S129N
- added F16, H23: 74LS08, symbol 74xx:74LS08
- added F18, F19, F2: 74LS157, symbol jt74:74LS157
- added F20, G20: 74LS399, symbol 74xx:74LS399
- added G19: 74LS367, symbol 74xx:74LS367
- added H16: 74LS04, symbol jt74:74LS04
- added unit 1 of H18
- added H19: 74LS74, symbol jt74:74LS74
- added I20: 74LS175, symbol 74xx:74LS175
- added unit 1 of J16 (x2)
- added unit 6 of J16
- added unit 5 of J16
- added RA4.7KX6: R_Network06_US, Resistor_THT:R_Array_SIP7, symbol Device:R_Network06_US
Connections:
- net MAIN_A1: now also F18.2 (I0a)
- net MAIN_A10: now also F2.5 (I0b)
- net MAIN_A2: now also F18.5 (I0b)
- net MAIN_A3: now also F18.11 (I0c)
- net MAIN_A4: now also F18.14 (I0d)
- net MAIN_A5: now also F19.2 (I0a)
- net MAIN_A6: now also F19.5 (I0b)
- net MAIN_A7: now also F19.11 (I0c)
- net MAIN_A8: now also F19.14 (I0d)
- net MAIN_A9: now also F2.2 (I0a)
- net VCC: now also H18.13 (~{R}), H20.1 (~{Mr}), I21.1 (~{Mr}), J21.1 (~{Mr}), E20.16 (VCC), F20.16 (VCC), H18.4 (~{S}), H19.1 (~{R}), H19.13 (~{R}), H19.4 (~{S}), I20.1 (~{Mr})
- net VSS: now also H21.8 (GND), J20.8 (GND), E14.18 (~{CS}), E14.19 (A10), E20.8 (VSS), F18.15 (~{G}), F19.15 (~{G}), F2.15 (~{G}), F20.8 (GND), G20.11 (I0c), G20.14 (I0d), RA4.7KX6.1 (common)
- net OBJOE: now reaches I19.1 (OEa)
- net OBJOE: now also I19.19 (OEb)
- net M12B: now reaches I21.9 (Cp)
- net M12B: now also J21.9 (Cp), H16.3, H19.11 (C), J16.12
- net CLK2: now reaches H20.11 (Cp)
- net CLK2: now also F20.9 (CP), G20.9 (CP), H19.3 (C), J16.1
- net at H20.12 (Q4): now also G19.12 (I5)
- net at H20.15 (Q5): now also G19.14 (I6)
- net at H20.2 (Q0): now also G19.2 (I1)
- net at H20.5 (Q1): now also G19.4 (I2)
- net at H20.6 (Q2): now also G19.6 (I3)
- net at H20.9 (Q3): now also G19.10 (I4)
- net CA20: now reaches I24.10 (CA20)
- net CA20: now also J20.4 (D0)
- net CA19: now reaches I24.11 (CA19)
- net CLK1: now reaches I24.2 (M12)
- net VSCM: now reaches I24.59 (VSCN)
- net VSCM: now also I20.10 (Q2)
- net HSCM: now reaches I24.60 (HSCM)
- net HSCM: now also I20.15 (Q3)
- net VRC: now reaches I24.61 (VRC)
- net VRC: now also I20.3 (~{Q0})
- net HRC: now reaches I24.62 (HRC)
- net HRC: now also I20.6 (~{Q1})
- net CA23: now reaches I24.7 (CA23)
- net CA22: now reaches I24.8 (CA22)
- net CA21: now reaches I24.9 (CA21)
- net CA21: now also J20.5 (D1)
- net at H18.10 (~{S}): now also H18.1 (~{R}), H19.10 (~{S}), J16.10
- net at H18.11 (C), J20.9 (Cp): now also H21.9 (CP), I20.9 (Cp), J16.2
- net ~{AS}: now reaches H18.12 (D)
- net ~{AS}: now also J16.11
- net at H18.9 (Q): now also F16.5
- net ~{RCS0}: now reaches J20.1 (~{Mr})
- net at J20.14 (~{Q3}): now also H19.2 (D)
- new net: J16.13, J16.2
- new net: H18.2 (D), H23.3
- new net: F18.10 (I1c), F20.10 (Qc)
- new net: E14.6 (A2), F18.12 (Zd)
- new net: F18.13 (I1d), F20.15 (Qd)
- new net: F18.3 (I1a), F20.2 (Qa)
- new net: E14.4 (A4), F18.4 (Za)
- new net: F18.6 (I1b), F20.7 (Qb)
- new net: E14.2 (A6), F18.7 (Zb)
- new net: E14.1 (A7), F18.9 (Zc)
- new net: F16.4, H18.6 (~{Q})
- new net: F16.6, H19.12 (D)
- new net: H16.4, H18.3 (C)
- new net: F19.10 (I1c), G20.10 (Qc)
- new net: E14.8 (A0), F19.12 (Zd)
- new net: F19.13 (I1d), G20.15 (Qd)
- new net: F19.3 (I1a), G20.2 (Qa)
- new net: E14.23 (A8), F19.4 (Za)
- new net: F19.6 (I1b), G20.7 (Qb)
- new net: E14.7 (A1), F19.7 (Zb)
- new net: E14.22 (A9), F19.9 (Zc)
- new net: F16.2, H19.9 (Q)
- new net: E14.20 (~{OE}), F2.9 (Zc)
- new net: E14.3 (A5), F2.4 (Za)
- new net: E14.5 (A3), F2.7 (Zb)
- new net: G19.1 (OEa), G19.15 (OEb), H19.5 (Q)
- new net: G19.11 (O5b), G20.3 (I0a), RA4.7KX6.6 (R5)
- new net: G19.13 (O6b), G20.6 (I0b), RA4.7KX6.7 (R6)
- new net: F20.3 (I0a), G19.3 (O1a), RA4.7KX6.2 (R1)
- new net: F20.6 (I0b), G19.5 (O2a), RA4.7KX6.3 (R2)
- new net: F20.11 (I0c), G19.7 (O3a), RA4.7KX6.4 (R3)
- new net: F20.14 (I0d), G19.9 (O4a), RA4.7KX6.5 (R4)
- new net: E18.1 (A->B), F2.11 (I0c)
- new net 63S: E20.12 (D1), F20.1 (S), G20.1 (S)
- new net CLK4: J16.1
- new net OBJSE: F16.1, F18.1 (SEL), F19.1 (SEL)
- new net PAL14: H23.2
- new net PAL17: H23.1
- new net ~{HBK}: I20.13 (D3)
- new net ~{HSYNC}: I20.5 (D1)
- new net ~{VBK}: I20.12 (D2)
- new net ~{VSYNC}: I20.4 (D0)
- no-connect marks 6 -> 13
Other:
- moved on the sheet: D23, F23, G16B, H18B, H20, H21, I19, I21, I24, J16C, J20, J21

Commit message: wip rollerg sch: PSAC
Parts:
- removed RA4.7KX6: R_Network06_US, Resistor_THT:R_Array_SIP7, symbol Device:R_Network06_US
- added E16: 74LS245, symbol jt74:74LS245
- added RA4.7KX1: R_Network06_US, Resistor_THT:R_Array_SIP7, symbol Device:R_Network06_US
- renumbered F2 to E19
Connections:
- net 63S is gone; now on net 63S1: E20.12 (D1), F20.1 (S), G20.1 (S)
- net DB0: now also E18.2 (A0); no longer I19.18 (O0a)
- net DB1: now also E18.3 (A1); no longer I19.16 (O1a)
- net DB2: now also E18.4 (A2); no longer I19.14 (O2a)
- net DB3: now also E18.5 (A3); no longer I19.12 (O3a)
- net DB4: now also E18.6 (A4); no longer I19.9 (O0b)
- net DB5: now also E18.7 (A5); no longer I19.7 (O1b)
- net DB6: now also E18.8 (A6); no longer I19.5 (O2b)
- net DB7: now also E18.9 (A7); no longer I19.3 (O3b)
- net OBJSE: now also E19.1 (SEL)
- net VCC: now also E14.24 (VCC), G20.16 (VCC)
- net VSS: now also E14.12 (VSS), E19.10 (I1c), E19.6 (I1b), E20.13 (~{CE}1), E20.14 (~{CE}2), G20.8 (GND), RA4.7KX1.1 (common)
- net POBJ2: now reaches F18.10 (I1c), F20.10 (Qc)
- net COLA2: now reaches E14.6 (A2), F18.12 (Zd)
- net POBJ3: now reaches F18.13 (I1d), F20.15 (Qd)
- net POBJ0: now reaches F18.3 (I1a), F20.2 (Qa)
- net COLA4: now reaches E14.4 (A4), F18.4 (Za)
- net POBJ1: now reaches F18.6 (I1b), F20.7 (Qb)
- net COLA6: now reaches E14.2 (A6), F18.7 (Zb)
- net COLA7: now reaches E14.1 (A7), F18.9 (Zc)
- net POBJ6: now reaches F19.10 (I1c), G20.10 (Qc)
- net COLA0: now reaches E14.8 (A0), F19.12 (Zd)
- net POBJ7: now reaches F19.13 (I1d), G20.15 (Qd)
- net POBJ4: now reaches F19.3 (I1a), G20.2 (Qa)
- net COLA8: now reaches E14.23 (A8), F19.4 (Za)
- net POBJ5: now reaches F19.6 (I1b), G20.7 (Qb)
- net COLA1: now reaches E14.7 (A1), F19.7 (Zb)
- net COLA9: now reaches E14.22 (A9), F19.9 (Zc)
- net DTAC: now reaches F16.3
- net COLAR1: now reaches E14.10 (D1)
- net COLAR1: now also E18.17 (B1)
- net COLAR2: now reaches E14.11 (D2)
- net COLAR2: now also E18.16 (B2)
- net COLAR3: now reaches E14.13 (D3)
- net COLAR3: now also E18.15 (B3)
- net COLAR4: now reaches E14.14 (D4)
- net COLAR4: now also E18.14 (B4)
- net COLAR5: now reaches E14.15 (D5)
- net COLAR5: now also E18.13 (B5)
- net COLAR6: now reaches E14.16 (D6)
- net COLAR6: now also E18.12 (B6)
- net COLAR7: now reaches E14.17 (D7)
- net COLAR7: now also E18.11 (B7)
- net POE: now reaches E14.20 (~{OE}), E19.9 (Zc)
- net WR: now reaches E14.21 (~{WR})
- net COLA5: now reaches E14.3 (A5), E19.4 (Za)
- net COLA3: now reaches E14.5 (A3), E19.7 (Zb)
- net COLAR0: now reaches E14.9 (D0)
- net COLAR0: now also E18.18 (B0)
- net VD3: now reaches G19.10 (I4), H20.9 (Q3)
- net VDR5: now reaches G19.11 (O5b), G20.3 (I0a)
- net VDR5: now also RA4.7KX1.6 (R5)
- net VD4: now reaches G19.12 (I5), H20.12 (Q4)
- net VDR6: now reaches G19.13 (O6b), G20.6 (I0b)
- net VDR6: now also RA4.7KX1.7 (R6)
- net VD5: now reaches G19.14 (I6), H20.15 (Q5)
- net VD0: now reaches G19.2 (I1), H20.2 (Q0)
- net VDR1: now reaches F20.3 (I0a), G19.3 (O1a)
- net VDR1: now also E20.5 (A0), RA4.7KX1.2 (R1)
- net VD1: now reaches G19.4 (I2), H20.5 (Q1)
- net VDR2: now reaches F20.6 (I0b), G19.5 (O2a)
- net VDR2: now also E20.6 (A1), RA4.7KX1.3 (R2)
- net VD2: now reaches G19.6 (I3), H20.6 (Q2)
- net VDR3: now reaches F20.11 (I0c), G19.7 (O3a)
- net VDR3: now also E20.7 (A2), RA4.7KX1.4 (R3)
- net VDR4: now reaches F20.14 (I0d), G19.9 (O4a)
- net VDR4: now also E20.4 (A3), RA4.7KX1.5 (R4)
- net ~{RD}: now reaches E18.1 (A->B), E19.11 (I0c)
- net ~{RD}: now also E16.1 (A->B)
- net VD7: now reaches E19.3 (I1a)
- net VD7: now also H20.19 (Q7)
- net VD6: now reaches H20.16 (Q6)
- net 63S2: now reaches H20.17 (D6)
- net 63S2: now also E20.11 (D2)
- net 63S1: now reaches H20.18 (D7)
- net SDI0: now reaches E20.1 (A6)
- net G18P7: now reaches E20.15 (A7)
- net OBJPXL8: now reaches E20.2 (A5)
- net OBOK: now reaches E20.3 (A4)
- net OBJPXL6: now reaches G20.12 (I1c)
- net OBJPXL7: now reaches G20.13 (I1d)
- net OBJPXL4: now reaches G20.4 (I1a)
- net OBJPXL5: now reaches G20.5 (I1b)
- net OBJPXL2: now reaches F20.12 (I1c)
- net OBJPXL3: now reaches F20.13 (I1d)
- net OBJPXL0: now reaches F20.4 (I1a)
- net OBJPXL1: now reaches F20.5 (I1b)
- new net MAIN_Z0: I19.12 (O3a)
- new net MAIN_Z1: I19.14 (O2a)
- new net MAIN_Z2: I19.18 (O0a)
- new net MAIN_Z3: I19.16 (O1a)
- new net MAIN_Z4: I19.3 (O3b)
- new net MAIN_Z5: I19.5 (O2b)
- new net MAIN_Z6: I19.9 (O0b)
- new net MAIN_Z7: I19.7 (O1b)
- no-connect marks 13 -> 15
Other:
- moved on the sheet: D23, E14, E18, E19, E20, F16A, F16B, F18, F19, F20, F23, G16B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

Commit message: wip rollerg sch: SOUND
Parts:
- added C13, C14: 74LS273, symbol 74xx:74LS273
- added D18: 74LS32, symbol jt74:74LS32
- added E15: SRAM2K8B, symbol jt_ram:SRAM2K8B
- added E16: 74LS245, symbol jt74:74LS245
- added F7: 74LS04, symbol jt74:74LS04
- renumbered J16 to H16
Connections:
- net CA19: now also D23.24 (~{OE}), F7.13
- net CLK4: now also I24.63 (M6)
- net COLA0: now also E15.6 (A2)
- net COLA1: now also E15.5 (A3)
- net COLA2: now also E15.4 (A4)
- net COLA3: now also E15.3 (A5)
- net COLA4: now also E15.2 (A6)
- net COLA5: now also E15.22 (A9)
- net COLA6: now also E15.23 (A8)
- net COLA7: now also E15.1 (A7)
- net COLA8: now also E15.8 (A0)
- net COLA9: now also E15.7 (A1)
- net COLAR0: now also C13.3 (D0)
- net COLAR1: now also C13.4 (D1)
- net COLAR2: now also C13.7 (D2)
- net COLAR3: now also C13.8 (D3)
- net COLAR4: now also C13.13 (D4)
- net COLAR5: now also C13.14 (D5)
- net COLAR6: now also C13.17 (D6)
- net COLAR7: now also C13.18 (D7)
- net DB0: now also E16.2 (A0)
- net DB1: now also E16.3 (A1)
- net DB2: now also E16.4 (A2)
- net DB3: now also E16.5 (A3)
- net DB4: now also E16.6 (A4)
- net DB5: now also E16.7 (A5)
- net DB6: now also E16.8 (A6)
- net DB7: now also E16.9 (A7)
- net MAIN_A0: now also D18.5
- net OBJSE: now also D18.1, D18.4
- net POE: now also E15.20 (~{OE})
- net VCC: now also G19.16 (VCC), H20.20 (VCC), H21.16 (VCC), I19.20 (VCC), I21.16 (VCC), J21.16 (VCC), C13.20 (VCC), C14.20 (VCC), E15.24 (VCC)
- net VSS: now also D23.22 (~{CE}), F23.22 (~{CE}), G19.8 (GND), H20.10 (GND), I19.10 (GND), I20.8 (GND), I21.8 (GND), J21.8 (GND), C13.10 (GND), C14.10 (GND), E15.12 (VSS), E15.18 (~{CS}), E15.19 (A10)
- net ~{RD}: now also E16.1 (A->B)
- net ~{CA19}: now reaches F23.24 (~{OE})
- net ~{CA19}: now also D18.2, F7.12
- net ~{CLK2}: now reaches H16.13, H16.2
- net at E16.19 (~{CE}): now also D18.3
- net at E18.19 (~{CE}): now also D18.6
- new net: C13.1 (~{Mr}), C14.1 (~{Mr})
- new net: C13.11 (Cp), C14.11 (Cp)
- no-connect marks 15 -> 19
Other:
- moved on the sheet: E16, H16A, H16F

Commit message: wip rollerg sch: CABINET AND RGB
Parts:
- removed C13, C14: 74LS273, symbol 74xx:74LS273
- removed D18: 74LS32, symbol jt74:74LS32
- removed E14, E15: SRAM2K8B, symbol jt_ram:SRAM2K8B
- removed E16 (x2), E18: 74LS245, symbol jt74:74LS245
- removed E19, F18, F19: 74LS157, symbol jt74:74LS157
- removed F7: 74LS04, symbol jt74:74LS04
Connections:
- no-connect marks 19 -> 22
Other:
- added sheet RGB (RGB.kicad_sch)

Commit message: almost complete rollerg sch
Connections:
- net MAIN_Z0 is gone; now on net DB3: I19.12 (O3a)
- net MAIN_Z1 is gone; now on net DB2: I19.14 (O2a)
- net MAIN_Z2 is gone; now on net DB0: I19.18 (O0a)
- net MAIN_Z3 is gone; now on net DB1: I19.16 (O1a)
- net MAIN_Z4 is gone; now on net DB7: I19.3 (O3b)
- net MAIN_Z5 is gone; now on net DB6: I19.5 (O2b)
- net MAIN_Z6 is gone; now on net DB4: I19.9 (O0b)
- net MAIN_Z7 is gone; now on net DB5: I19.7 (O1b)
- net VCC: now also I20.16 (VCC), J20.16 (VCC)
- net +5V: now reaches I24.32 (+5V)
- net +5V: now also I24.64 (+5V)
- net OBJPXL8 renamed OBOB
- net ~{RCS0} renamed RES
- no-connect marks 22 -> 26
Other:
- sheet RGB ports: added BLUE, CLK2, GREEN, MAIN_A0, MAIN_A[10..0], OBCE, OBJSE, POBJ[7..0], RED, VD7, WR, ~{CA19}, ~{DS}, ~{HBK}, ~{RD}, ~{VBK}; removed none
